File: MP4GS_PWR/MP4GS_Power.brd (EAGLE design)
At the start: 48.3 x 31.7 mm, 5 parts

Commit message: MP4GS_PWR revisions
still a WIP
Routing:
- net N$2: track 0.00 -> 22.1 mm
- net N$3: track 0.00 -> 17.1 mm
- net N$1: track 0.00 -> 12.0 mm
Other:
- board text added: "MP4GS-ARD-PWD"
- board text removed: "MP4GS Arduino PowerBoard r/0.5"

Commit message: WIP MP4GS_PWR
Connections:
- net GND: now also JP1.2, JP2.4

Commit message: Finalized MP4GS PWR board
Parts:
- added JP3: (no value), Haddock:1X02
Connections:
- net N$2: now also JP3.PLFT
Routing:
- net N$2: track 22.1 -> 28.5 mm
Other:
- board text added: "MP4GS Arduino PowerBoard r/0.5"
- board text removed: "MP4GS-ARD-PWD"
