File: MP4GS_PWR/MP4GS_Power.sch (EAGLE design)
At the start: 5 parts

Commit message: WIP MP4GS_PWR
Connections:
- net GND: now also JP1.2, JP2.4
Changed lines of the file:
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@@
 <segment>
 <pinref part="GND3" gate="1" pin="GND"/>
-<wire x1="30.48" y1="175.26" x2="30.48" y2="190.5" width="0.1524" layer="91"/>
+<wire x1="30.48" y1="175.26" x2="30.48" y2="177.8" width="0.1524" layer="91"/>
 <pinref part="JP1" gate="A" pin="4"/>
+<wire x1="30.48" y1="177.8" x2="30.48" y2="190.5" width="0.1524" layer="91"/>
 <wire x1="22.86" y1="175.26" x2="30.48" y2="175.26" width="0.1524" layer="91"/>
+<pinref part="JP1" gate="A" pin="2"/>
+<wire x1="22.86" y1="177.8" x2="30.48" y2="177.8" width="0.1524" layer="91"/>
+<junction x="30.48" y="177.8"/>
 </segment>
 <segment>
 <pinref part="GND2" gate="1" pin="GND"/>
 <wire x1="88.9" y1="144.78" x2="109.22" y2="144.78" width="0.1524" layer="91"/>
-<wire x1="109.22" y1="144.78" x2="109.22" y2="177.8" width="0.1524" layer="91"/>
+<wire x1="109.22" y1="144.78" x2="109.22" y2="175.26" width="0.1524" layer="91"/>
 <pinref part="JP2" gate="A" pin="2"/>
+<wire x1="109.22" y1="175.26" x2="109.22" y2="177.8" width="0.1524" layer="91"/>
 <wire x1="101.6" y1="177.8" x2="109.22" y2="177.8" width="0.1524" layer="91"/>
+<pinref part="JP2" gate="A" pin="4"/>
+<wire x1="101.6" y1="175.26" x2="109.22" y2="175.26" width="0.1524" layer="91"/>
+<junction x="109.22" y="175.26"/>
 </segment>
 <segment>

Commit message: Finalized MP4GS PWR board
Parts:
- added JP3: (no value), Haddock:PINHD-1X2
Connections:
- net N$2: now also JP3.1
Changed lines of the file:
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@@
 <part name="R1" library="rcl" deviceset="R-EU_" device="0207/10"/>
 <part name="GND4" library="supply1" deviceset="GND" device=""/>
+<part name="JP3" library="Haddock" deviceset="PINHD-1X2" device=""/>
 </parts>
 <sheets>
@@
 <instance part="R1" gate="G$1" x="66.04" y="129.54" rot="R90"/>
 <instance part="GND4" gate="1" x="66.04" y="111.76"/>
+<instance part="JP3" gate="G$1" x="127" y="182.88"/>
 </instances>
 <busses>
@@
 <wire x1="101.6" y1="175.26" x2="109.22" y2="175.26" width="0.1524" layer="91"/>
 <junction x="109.22" y="175.26"/>
+<wire x1="127" y1="182.88" x2="132.08" y2="182.88" width="0.1524" layer="91"/>
+<wire x1="132.08" y1="182.88" x2="132.08" y2="175.26" width="0.1524" layer="91"/>
+<wire x1="132.08" y1="175.26" x2="109.22" y2="175.26" width="0.1524" layer="91"/>
 </segment>
 <segment>
@@
 <wire x1="66.04" y1="160.02" x2="66.04" y2="149.86" width="0.1524" layer="91"/>
 <junction x="66.04" y="160.02"/>
+<pinref part="JP3" gate="G$1" pin="1"/>
+<wire x1="124.46" y1="185.42" x2="88.9" y2="185.42" width="0.1524" layer="91"/>
+<wire x1="88.9" y1="185.42" x2="88.9" y2="175.26" width="0.1524" layer="91"/>
+<junction x="88.9" y="175.26"/>
 </segment>
 </net>
